Commit message: adding aruco and navigation to aruco

File: rl_fra2mo_description/urdf/camera_gazebo_macro.xacro (robot description, xacro)
@@ -7,5 +7,5 @@
       <parent link="${parent}"/>
       <child link="camera_link"/>
-      <origin xyz="0.090925 0.0 0.06670" rpy="0 0 0" />
+      <origin xyz="0.100925 0.0 0.07670" rpy="0 0 0" />
     </joint>
     <link name="camera_link">
@@ -27,22 +27,21 @@
     <gazebo reference="camera_link">
         <material>Gazebo/Red</material>
-        <sensor name="camera" type="camera">
-            <always_on>true</always_on>
-            <visualize>true</visualize>
-            <update_rate>10</update_rate>
-            <topic>camera/image_raw</topic>
-            <camera>
-                <horizontal_fov>1.089</horizontal_fov>
-                <image>
-                    <format>R8G8B8</format>
-                    <width>640</width>
-                    <height>480</height>
-                </image>
-                <clip>
-                    <near>0.05</near>
-                    <far>8.0</far>
-                </clip>
-            </camera>
-        </sensor>
+          <sensor name="camera" type="camera">
+              <camera>
+              <horizontal_fov>1.047</horizontal_fov>
+              <image>
+                  <width>320</width>
+                  <height>240</height>
+              </image>
+              <clip>
+                  <near>0.1</near>
+                  <far>100</far>
+              </clip>
+              </camera>
+              <always_on>1</always_on>
+              <update_rate>30</update_rate>
+              <visualize>true</visualize>
+              <topic>camera</topic>
+          </sensor>
     </gazebo>
   </xacro:macro>
